Commit message: urdf

File: x1/urdf/x1.urdf (robot description, URDF)
Before this commit: robot x1, 58 links, 57 joints
Joints:
- joint arm_l_wrist_a_ball_joint: type fixed -> revolute
- joint arm_l_wrist_a_loop_joint: type fixed -> revolute
- joint arm_l_wrist_b_ball_joint: type fixed -> revolute
- joint arm_l_wrist_b_loop_joint: type fixed -> revolute
- joint arm_l_wrist_motor_a_link_joint: type fixed -> revolute
- joint arm_l_wrist_motor_b_link_joint: type fixed -> revolute
- joint arm_r_wrist_a_ball_joint: type fixed -> revolute
- joint arm_r_wrist_a_loop_joint: type fixed -> revolute
- joint arm_r_wrist_b_ball_joint: type fixed -> revolute
- joint arm_r_wrist_b_loop_joint: type fixed -> revolute
- joint arm_r_wrist_motor_a_link_joint: type fixed -> revolute
- joint arm_r_wrist_motor_b_link_joint: type fixed -> revolute
- joint left_elbow_pitch_joint: type fixed -> revolute
- joint left_elbow_yaw_joint: type fixed -> revolute
- joint left_shoulder_pitch_joint: type fixed -> revolute
- joint left_shoulder_roll_joint: type fixed -> revolute
- joint left_shoulder_yaw_joint: type fixed -> revolute
- joint left_wrist_pitch_joint: type fixed -> revolute
- joint leg_l_toe_a_ball_joint: type fixed -> revolute
- joint leg_l_toe_a_link_joint: type fixed -> revolute
- joint leg_l_toe_a_loop_joint: type fixed -> revolute
- joint leg_l_toe_b_ball_joint: type fixed -> revolute
- joint leg_l_toe_b_link_joint: type fixed -> revolute
- joint leg_l_toe_b_loop_joint: type fixed -> revolute
- joint leg_r_toe_a_ball_joint: type fixed -> revolute
- joint leg_r_toe_a_link_joint: type fixed -> revolute
- joint leg_r_toe_a_loop_joint: type fixed -> revolute
- joint leg_r_toe_b_ball_joint: type fixed -> revolute
- joint leg_r_toe_b_link_joint: type fixed -> revolute
- joint leg_r_toe_b_loop_joint: type fixed -> revolute
- joint lumber_pitch_joint: type fixed -> revolute
- joint lumber_roll_joint: type fixed -> revolute
- joint lumber_yaw_joint: type fixed -> revolute
- joint right_elbow_pitch_joint: type fixed -> revolute
- joint right_elbow_yaw_joint: type fixed -> revolute
- joint right_shoulder_pitch_joint: type fixed -> revolute
- joint right_shoulder_roll_joint: type fixed -> revolute
- joint right_shoulder_yaw_joint: type fixed -> revolute
- joint right_wrist_pitch_joint: type fixed -> revolute
- joint waist_motor_a_ball_joint: type fixed -> revolute
- joint waist_motor_a_link_joint: type fixed -> revolute
- joint waist_motor_a_loop_joint: type fixed -> revolute
- joint waist_motor_b_ball_joint: type fixed -> revolute
- joint waist_motor_b_link_joint: type fixed -> revolute
- joint waist_motor_b_loop_joint: type fixed -> revolute

Commit message: urdf

File: x1/urdf/x1.urdf (robot description, URDF)
Before this commit: robot x1, 58 links, 57 joints
Links:
- added link left_wrist_roll_link, mass 0.370899; collision cylinder length=0.1 radius=0.02; visual mesh filename=../meshes/left_wrist_roll.STL
- added link right_wrist_roll_link, mass 0.370899; collision cylinder length=0.1 radius=0.02; visual mesh filename=../meshes/right_wrist_roll.STL
Joints:
- added joint left_wrist_roll_joint: type revolute, parent left_wrist_pitch, child left_wrist_roll_link, origin xyz=0 0 0 rpy=0 1.570796 0, axis 1 0 0, limit lower=-3.14 upper=3.14 effort=0 velocity=2
- added joint right_wrist_roll_joint: type revolute, parent right_wrist_pitch, child right_wrist_roll_link, origin xyz=0 0 0 rpy=0 1.570796 0, axis 1 0 0, limit lower=-3.14 upper=3.14 effort=10.0 velocity=2.0
- joint arm_l_wrist_a_ball_joint: axis 0 0 0 -> 0 -1 0; limit (none) -> lower=0.0 upper=0.254 effort=50 velocity=0.005; type revolute -> prismatic

Commit message: pinocchio

File: x1/urdf/x1.urdf (robot description, URDF)
Before this commit: robot x1, 58 links, 57 joints
Joints:
- joint arm_l_wrist_a_ball_joint: type revolute -> fixed
- joint arm_l_wrist_a_loop_joint: type revolute -> fixed
- joint arm_l_wrist_b_ball_joint: type revolute -> fixed
- joint arm_l_wrist_b_loop_joint: type revolute -> fixed
- joint arm_r_wrist_a_ball_joint: type revolute -> fixed
- joint arm_r_wrist_a_loop_joint: type revolute -> fixed
- joint arm_r_wrist_b_ball_joint: type revolute -> fixed
- joint arm_r_wrist_b_loop_joint: type revolute -> fixed
- joint leg_l_toe_a_ball_joint: type revolute -> fixed
- joint leg_l_toe_a_loop_joint: type revolute -> fixed
- joint leg_l_toe_b_ball_joint: type revolute -> fixed
- joint leg_l_toe_b_link_joint: type revolute -> fixed
- joint leg_l_toe_b_loop_joint: type revolute -> fixed
- joint leg_r_toe_a_ball_joint: type revolute -> fixed
- joint leg_r_toe_a_loop_joint: type revolute -> fixed
- joint leg_r_toe_b_ball_joint: type revolute -> fixed
- joint leg_r_toe_b_link_joint: type revolute -> fixed
- joint leg_r_toe_b_loop_joint: type revolute -> fixed
- joint waist_motor_a_ball_joint: type revolute -> fixed
- joint waist_motor_a_loop_joint: type revolute -> fixed
- joint waist_motor_b_ball_joint: type revolute -> fixed
- joint waist_motor_b_link_joint: type revolute -> fixed
- joint waist_motor_b_loop_joint: type revolute -> fixed
